File: 3-term/CSC202_LP_MSPM0G3507_3TERM_BREAKOUT/CSC202_LP_MSPM0G3507_3TERM_BREAKOUT.kicad_pcb (KiCad board)
At the start: 2 copper layers, 90 x 35 mm, 9 parts, among them J1 J_IN1/J_IN3, J2 J_IN4/J_IN2, J3 J_OUT1, J4 J_OUT3, J5 J_OUT4, J6 J_OUT2

Commit message: completed 2-term version
Parts:
- added LOGO1: LOGO, 01-Shared_Project_Footprints:MCC-Logo, F.Cu at (92.4, 83.9)
Other:
- board text added: "CSC-202 LP-MSPM0G3507 3-TERM-STRIP BREADBOARD BREAKOUT"
- board text removed: "MCC CSC-202 LP-MSPM0G3507 3-TERM-STRIP BREADBOARD BREAKOUT"
