File: hardware/pcb/kicad/dipsw-module/CSC202_DIPSW/CSC202_DIPSW.kicad_sch (KiCad schematic)
At the start: 12 parts, among them J1 PWR-IN, J2 ADC-IF, J3 SW-IF, J4 MECH, SW1 ADC-EN, SW2 PB1, SW3 PB2, SW4 PB3, SW5 PB4, SW6 SW_DIP_x04

Commit message: add DIP switch module KiCad design
Other:
- company: (none) -> Eli Bell
- title: (none) -> CSC_202_SW_MODULE
Changed lines of the file:
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@@
 	(paper "A4")
 	(title_block
+		(title "CSC_202_SW_MODULE")
+		(company "Eli Bell")
 		(comment 3 "configurable analog input using a potentiometer with DIP-selectable ADC connection.")
 		(comment 4 "Four GPIO inputs with dual control via DIP switches and pushbuttons. Includes a")
